Commit message: Interia & Odom Improved

File: urdf/differential_drive.xacro (robot description, xacro)
@@ -8,7 +8,7 @@
 <link name="base_link">
   <inertial>
-    <origin rpy="0 0 0" xyz="-0.040010469235296664 9.471423530512231e-18 0.0050000000000195"/>
-    <mass value="0.09422466150306563"/>
-    <inertia ixx="0.0000794" ixy="-0.0" ixz="0.0" iyy="0.0001139" iyz="0.0" izz="0.0001916"/>
+    <origin rpy="0 0 0" xyz="-0.050010469235296664 9.471423530512231e-18 0.0050000000000195"/>
+    <mass value="1.0"/>
+    <inertia ixx="0.0012083" ixy="-0.0" ixz="0.0" iyy="0.0010167" iyz="0.0" izz="0.0022083"/>
   </inertial>
   <visual>
@@ -28,7 +28,7 @@
 <link name="left_wheel_1">
   <inertial>
-    <origin rpy="0 0 0" xyz="-1.1920926745734306e-09 -0.007500000000000007 7.450615905485458e-11"/>
-    <mass value="0.09803750446346561"/>
-    <inertia ixx="1.4e-05" ixy="0.0" ixz="-0.0" iyy="2.3e-05" iyz="-0.0" izz="1.4e-05"/>
+    <origin rpy="0 0 0" xyz="-1.1920926745734306e-09 0.009 7.450615905485458e-11"/>
+    <mass value="0.25"/>
+    <inertia ixx="0.000034514" ixy="0.0" ixz="-0.0" iyy="0.000059653" iyz="-0.0" izz="0.000034514"/>
   </inertial>
   <visual>
@@ -48,7 +48,7 @@
 <link name="right_wheel_1">
   <inertial>
-    <origin rpy="0 0 0" xyz="-1.1920926051844916e-09 0.007500000000000007 7.450545042031465e-11"/>
-    <mass value="0.09803750446346572"/>
-    <inertia ixx="1.4e-05" ixy="0.0" ixz="0.0" iyy="2.3e-05" iyz="-0.0" izz="1.4e-05"/>
+    <origin rpy="0 0 0" xyz="-1.1920926051844916e-09 -0.009 7.450545042031465e-11"/>
+    <mass value="0.25"/>
+    <inertia ixx="0.000034514" ixy="0.0" ixz="-0.0" iyy="0.000059653" iyz="-0.0" izz="0.000034514"/>
   </inertial>
   <visual>
@@ -69,6 +69,6 @@
   <inertial>
     <origin rpy="0 0 0" xyz="0.0 -5.039195081648916e-18 -0.0056390049196538596"/>
-    <mass value="0.055343764086740264"/>
-    <inertia ixx="3e-06" ixy="0.0" ixz="0.0" iyy="3e-06" iyz="0.0" izz="5e-06"/>
+    <mass value="0.1"/>
+    <inertia ixx="0.000005826" ixy="0.0" ixz="0.0" iyy="0.000005814" iyz="0.0" izz="0.000008983"/>
   </inertial>
   <visual>
